File: super_expander.kicad_pcb (KiCad board)
At the start: 4 copper layers, 100 x 100 mm, 336 parts, among them J1 PA, J10 PK, J11 PM, J12 PO, J13 PJ, J14 PL, J15 PN, J16 PP, J17 PQ, J18 PS, J19 PU, J2 PC, J20 PW, J21 PR, J22 PT, J23 PV, J24 PX, J25 PY, J26 PAA, J27 PAC, J28 PAE, J29 PZ, J3 PE, J30 PAB, J31 PAD, J32 PAF, J33 PAG, J34 PAI, J35 PAK, J36 PAM, J37 PAH, J38 PAJ, J39 PAL, J4 PG, J40 PAN, J41 PAO, J42 PAQ, J43 PAS, J44 PAU, J45 PAP, J46 PAR, J47 PAT, J48 PAV, J49 PAW, J5 PB, J50 PAY, J51 PBA, J52 PBC, J53 PAX, J54 PAZ, J55 PBB, J56 PBD, J57 PBE, J58 PBG, J59 PBI, J6 PD, J60 PBK, J61 PBF, J62 PBH, J63 PBJ, J64 PBL, J7 PF, J8 PH, J9 PI, SW1 MCU_RESET, U1 AW9523B, U10 AW9523B, U11 AW9523B, U12 AW9523B, U13 AW9523B, U14 AW9523B, U15 AW9523B, U16 AW9523B, U17 AW9523B, U18 AW9523B, U19 AW9523B, U2 AW9523B, U20 AW9523B, U21 AW9523B, U22 AW9523B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

Commit message: Continue Routing
Parts:
- added C35: 100nF, Capacitor_SMD:C_0603_1608Metric, F.Cu at (56.6, 78.3)
- added C36: 100nF, Capacitor_SMD:C_0603_1608Metric, F.Cu at (61.4, 78.3)
- added C37: 100nF, Capacitor_SMD:C_0603_1608Metric, F.Cu at (138.9, 78.3)
- added C38: 100nF, Capacitor_SMD:C_0603_1608Metric, F.Cu at (143.7, 78.3)
- added C41: 100uF, Capacitor_THT:CP_Radial_D6.3mm_P2.50mm, F.Cu at (132.6, 78.2)
- added C42: 100uF, Capacitor_THT:CP_Radial_D6.3mm_P2.50mm, F.Cu at (89.8, 67.2)
- added D1: 1N5819, Diode_SMD:D_SOD-123F, F.Cu at (61.3, 62.9)
- added D2: 0603ESDA-05N, Diode_SMD:D_0603_1608Metric, F.Cu at (61.7, 67.1)
- added D3: 0603ESDA-05N, Diode_SMD:D_0603_1608Metric, F.Cu at (61.7, 70.4)
- added D4: LED_I2C, LED_SMD:LED_0603_1608Metric, F.Cu at (69.9, 64.0)
- added D5: ZMM6V2, Diode_SMD:D_MiniMELF, F.Cu at (122.8, 67.4)
- added FB1: FCM1608KF-121T05, Inductor_SMD:L_0603_1608Metric, F.Cu at (57.3, 64.8)
- added FB2: FCM1608KF-121T05, Inductor_SMD:L_0603_1608Metric, F.Cu at (57.3, 71.1)
- added G***: LOGO, sleepyLogo:sleepylogo_20mm, F.Cu at (73.2, 81.0)
- added J65: USB_B_Micro, Connector_USB:USB_Micro-B_Molex_47346-0001, F.Cu at (52.7, 67.1)
- added J66: I2C Passthrough, Connector_PinHeader_2.54mm:PinHeader_1x05_P2.54mm_Vertical, F.Cu at (52.5, 78.0)
- added J67: I2C Passthrough, Connector_PinHeader_2.54mm:PinHeader_1x05_P2.54mm_Vertical, F.Cu at (147.8, 78.1)
- added J68: Barrel_Jack_Switch, Connector_BarrelJack:BarrelJack_Horizontal, F.Cu at (135.6, 69.8)
- added JP4: I2C BUF PASS, Resistor_SMD:R_0402_1005Metric, F.Cu at (59.0, 81.1)
- added JP5: I2C BUF PASS, Resistor_SMD:R_0402_1005Metric, F.Cu at (141.3, 81.1)
- added JP6: I2C BUF PASS, Resistor_SMD:R_0402_1005Metric, F.Cu at (59.0, 82.5)
- added JP7: I2C BUF PASS, Resistor_SMD:R_0402_1005Metric, F.Cu at (141.3, 82.5)
- added Q1: IRF7410, Package_SO:SOIC-8_3.9x4.9mm_P1.27mm, F.Cu at (128.6, 67.4)
- added R1: 1k, Resistor_SMD:R_0603_1608Metric, F.Cu at (69.9, 62.3)
- added R2: 100k, Resistor_SMD:R_0603_1608Metric, F.Cu at (120.0, 66.3)
- added U35: MCP2221A-I/ST, Package_SO:TSSOP-14_4.4x5mm_P0.65mm, F.Cu at (72.0, 67.8)
- added U36: TCA9517, Package_SO:VSSOP-8_3.0x3.0mm_P0.65mm, F.Cu at (59.0, 81.8)
- added U37: TCA9517, Package_SO:VSSOP-8_3.0x3.0mm_P0.65mm, F.Cu at (141.3, 81.8)
- SW1: footprint Button_Switch_THT:SW_PUSH_6mm -> super_expander:TS-1101
- moved C16 109.5 mm to (65.8, 64.0), turned to 180 degrees
- moved RN4 106.7 mm to (104.0, 67.1)
- moved RN3 106.7 mm to (104.0, 82.9)
- moved U34 106.7 mm to (100.3, 75.0)
- moved JP2 106.6 mm to (88.8, 81.2)
- moved JP3 106.6 mm to (84.7, 81.2)
- moved JP1 106.6 mm to (92.9, 81.2)
- moved RN5 105.9 mm to (99.2, 67.1)
- moved RN2 105.9 mm to (99.2, 82.9)
- moved C15 98.4 mm to (72.0, 72.8), turned to 180 degrees
- moved C34 86.9 mm to (94.7, 72.2), turned to 90 degrees
- moved RN1 85.8 mm to (113.6, 69.7)
- moved SW1 79.0 mm to (116.5, 81.4)
- moved U33 77.7 mm to (113.5, 75.0), turned to 180 degrees
- moved C33 73.4 mm to (109.8, 80.0), turned to 270 degrees
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- renumbered C35 to C39, C36 to C40
Connections:
- C16 pad 1: +5V -> Net-(C16-Pad1)
- C19 pad 1: +5V -> Net-(C16-Pad1)
- C20 pad 1: +5V -> Net-(C16-Pad1)
- RN1 pad 1: Net-(RN1-Pad1) -> SDA
- RN1 pad 3: Net-(RN1-Pad3) -> SCL
- RN1 pad 4: Net-(RN1-Pad4) -> ~MRST
- SW1 pad 1: Net-(RN1-Pad1) -> ~MRST
- U1 pad 19: /Block0to3/SCL0 -> /SCL0
- U1 pad 20: /Block0to3/SDA0 -> /SDA0
- U10 pad 19: /Block0to3/SCL2 -> /SCL2
- U10 pad 20: /Block0to3/SDA2 -> /SDA2
- U11 pad 19: /Block0to3/SCL2 -> /SCL2
- U11 pad 20: /Block0to3/SDA2 -> /SDA2
- U12 pad 19: /Block0to3/SCL2 -> /SCL2
- U12 pad 20: /Block0to3/SDA2 -> /SDA2
- U13 pad 19: /Block0to3/SCL3 -> /SCL3
- U13 pad 20: /Block0to3/SDA3 -> /SDA3
- U14 pad 19: /Block0to3/SCL3 -> /SCL3
- U14 pad 20: /Block0to3/SDA3 -> /SDA3
- U15 pad 19: /Block0to3/SCL3 -> /SCL3
- U15 pad 20: /Block0to3/SDA3 -> /SDA3
- U16 pad 19: /Block0to3/SCL3 -> /SCL3
- U16 pad 20: /Block0to3/SDA3 -> /SDA3
- U17 pad 19: /Block4to7/SCL4 -> /SCL4
- U17 pad 20: /Block4to7/SDA4 -> /SDA4
- U18 pad 19: /Block4to7/SCL4 -> /SCL4
- U18 pad 20: /Block4to7/SDA4 -> /SDA4
- U19 pad 19: /Block4to7/SCL4 -> /SCL4
- U19 pad 20: /Block4to7/SDA4 -> /SDA4
- U2 pad 19: /Block0to3/SCL0 -> /SCL0
- U2 pad 20: /Block0to3/SDA0 -> /SDA0
- U20 pad 19: /Block4to7/SCL4 -> /SCL4
- U20 pad 20: /Block4to7/SDA4 -> /SDA4
- U21 pad 19: /Block4to7/SCL5 -> /SCL5
- U21 pad 20: /Block4to7/SDA5 -> /SDA5
- U22 pad 19: /Block4to7/SCL5 -> /SCL5
- U22 pad 20: /Block4to7/SDA5 -> /SDA5
- U23 pad 19: /Block4to7/SCL5 -> /SCL5
- U23 pad 20: /Block4to7/SDA5 -> /SDA5
- U24 pad 19: /Block4to7/SCL5 -> /SCL5
- U24 pad 20: /Block4to7/SDA5 -> /SDA5
- U25 pad 19: /Block4to7/SCL6 -> /SCL6
- U25 pad 20: /Block4to7/SDA6 -> /SDA6
- U26 pad 19: /Block4to7/SCL6 -> /SCL6
- U26 pad 20: /Block4to7/SDA6 -> /SDA6
- U27 pad 19: /Block4to7/SCL6 -> /SCL6
- U27 pad 20: /Block4to7/SDA6 -> /SDA6
- U28 pad 19: /Block4to7/SCL6 -> /SCL6
- U28 pad 20: /Block4to7/SDA6 -> /SDA6
- U29 pad 19: /Block4to7/SCL7 -> /SCL7
- U29 pad 20: /Block4to7/SDA7 -> /SDA7
- U3 pad 19: /Block0to3/SCL0 -> /SCL0
- U3 pad 20: /Block0to3/SDA0 -> /SDA0
- U30 pad 19: /Block4to7/SCL7 -> /SCL7
- U30 pad 20: /Block4to7/SDA7 -> /SDA7
- U31 pad 19: /Block4to7/SCL7 -> /SCL7
- U31 pad 20: /Block4to7/SDA7 -> /SDA7
- U32 pad 19: /Block4to7/SCL7 -> /SCL7
- U32 pad 20: /Block4to7/SDA7 -> /SDA7
- U33 pad 1: Net-(RN1-Pad1) -> ~MRST
- U33 pad 5: Net-(RN1-Pad3) -> SDA
- U33 pad 7: Net-(RN1-Pad4) -> SCL
- U34 pad 22: Net-(RN1-Pad4) -> SCL
- U34 pad 23: Net-(RN1-Pad3) -> SDA
- U4 pad 19: /Block0to3/SCL0 -> /SCL0
- U4 pad 20: /Block0to3/SDA0 -> /SDA0
- U5 pad 19: /Block0to3/SCL1 -> /SCL1
- U5 pad 20: /Block0to3/SDA1 -> /SDA1
- U6 pad 19: /Block0to3/SCL1 -> /SCL1
- U6 pad 20: /Block0to3/SDA1 -> /SDA1
- U7 pad 19: /Block0to3/SCL1 -> /SCL1
- U7 pad 20: /Block0to3/SDA1 -> /SDA1
- U8 pad 19: /Block0to3/SCL1 -> /SCL1
- U8 pad 20: /Block0to3/SDA1 -> /SDA1
- U9 pad 19: /Block0to3/SCL2 -> /SCL2
- U9 pad 20: /Block0to3/SDA2 -> /SDA2
Routing:
- net ~RST: track 346.0 -> 901.2 mm, vias 2 -> 39
- net SCL: track 0.00 -> 135.2 mm, vias 0 -> 6
- net SDA: track 0.00 -> 134.9 mm, vias 0 -> 6
- net /SDA4: track 0.00 -> 133.7 mm, vias 0 -> 7
- net /SCL4: track 0.00 -> 132.2 mm, vias 0 -> 5
- net /SDA3: track 0.00 -> 125.6 mm, vias 0 -> 5
- net /SCL7: track 0.00 -> 122.3 mm, vias 0 -> 5
- net /SCL3: track 0.00 -> 121.9 mm, vias 0 -> 9
- net /SDA7: track 0.00 -> 120.0 mm, vias 0 -> 5
- net /SDA0: track 0.00 -> 115.2 mm, vias 0 -> 9
- net /SCL0: track 0.00 -> 112.1 mm, vias 0 -> 5
- net /SCL5: track 0.00 -> 110.3 mm, vias 0 -> 1
- net /SDA5: track 0.00 -> 106.8 mm, vias 0 -> 9
- net /SCL6: track 0.00 -> 105.5 mm, vias 0 -> 5
- net /SDA2: track 0.00 -> 102.7 mm, vias 0 -> 5
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- added copper zone on B.Cu, net GND
- added copper zone on F.Cu, net GND
Other:
- net class Default: clearance 0.2 -> 0.14
- rule trace_clearance: 0.2 -> 0.14
- board text added: "0"
- board text added: "1"
- board text added: "3..0"
- board text added: "4..7"
- board text added: "A0"
- board text added: "A1"
- board text added: "A2"
- board text added: "JLCJLCJLCJLC"
- board text added: "PBE"
- board text added: "PBF"
- board text added: "Reset"
- board text added: "Super Expander:"
- board text added: "What if ATtiny85 has 512 I/O pins?"
- board text added: "www.sleepyponylabs.com"
