File: Block4to7.sch (KiCad schematic (older format))
At the start: 144 parts, among them J33 PAG, J34 PAI, J35 PAK, J36 PAM, J37 PAH, J38 PAJ, J39 PAL, J40 PAN, J41 PAO, J42 PAQ, J43 PAS, J44 PAU, J45 PAP, J46 PAR, J47 PAT, J48 PAV, J49 PAW, J50 PAY, J51 PBA, J52 PBC, J53 PAX, J54 PAZ, J55 PBB, J56 PBD, J57 PBE, J58 PBG, J59 PBI, J60 PBK, J61 PBF, J62 PBH, J63 PBJ, J64 PBL, U17 AW9523B, U18 AW9523B, U19 AW9523B, U20 AW9523B, U21 AW9523B, U22 AW9523B, U23 AW9523B, U24 AW9523B, U25 AW9523B, U26 AW9523B, U27 AW9523B, U28 AW9523B, U29 AW9523B, U30 AW9523B, U31 AW9523B, U32 AW9523B

Commit message: Continue Routing
Changed lines of the file:
@@
 Wire Bus Line
 	11350 1650 7550 1650
+Text Label 3550 1550 2    50   ~ 0
+SCL[0..7]
+Text Label 3550 1650 2    50   ~ 0
+SDA[0..7]
 $EndSCHEMATC

Commit message: Change some C and R values
Parts:
- RN100, RN101, RN102, RN103, RN104, RN105, RN106, RN107, RN108, RN109, RN110, RN111, RN112, RN113, RN114, RN115, RN116, RN117, RN118, RN119, RN120, RN121, RN122, RN123, RN124, RN125, RN126, RN127, RN128, RN129, RN130, RN131, RN132, RN133, RN70, RN71, RN72, RN73, RN74, RN75, RN76, RN77, RN78, RN79, RN80, RN81, RN82, RN83, RN84, RN85, RN86, RN87, RN88, RN89, RN90, RN91, RN92, RN93, RN94, RN95, RN96, RN97, RN98, RN99: value 1k -> 470
